File: KiCAD/OLED_Panel.sch (KiCad schematic (older format))
At the start: 9 parts

Commit message: Add STM32 base circuit for power control and USB, also a lot of other things
Connections:
- net +BATT: now reaches OEL601.5 (VBAT)
Changed lines of the file:
@@
 $Descr A4 11693 8268
 encoding utf-8
-Sheet 7 7
+Sheet 5 6
 Title ""
 Date ""
@@
 Wire Wire Line
 	5200 3375 5325 3375
+$Comp
+L power:+BATT #PWR?
+U 1 1 611DA85E
+P 5775 2625
+AR Path="/60EE6959/611DA85E" Ref="#PWR?"  Part="1"
+AR Path="/61017570/611DA85E" Ref="#PWR0152"  Part="1"
+F 0 "#PWR0152" H 5775 2475 50  0001 C CNN
+F 1 "+BATT" H 5790 2798 50  0000 C CNN
+F 2 "" H 5775 2625 50  0001 C CNN
+F 3 "" H 5775 2625 50  0001 C CNN
+	1    5775 2625
+	1    0    0    -1
+$EndComp
+Wire Wire Line
+	5775 2775 5775 2625
 $EndSCHEMATC

Commit message: Continue work on TapV2's schematic, almost completing it!
Parts:
- C603, C604: value 1uF 0603 16V -> 1uF 0402 16V; footprint Capacitor_SMD:C_0603_1608Metric -> Capacitor_SMD:C_0402_1005Metric
- C605, C607: value 2.2uF 0603 16V -> 2.2uF 0402 16V; footprint Capacitor_SMD:C_0603_1608Metric -> Capacitor_SMD:C_0402_1005Metric
Connections:
- net +3V3: now also OEL601.9 (~EN)
Changed lines of the file:
@@
 P 7525 4325
 F 0 "C607" V 7475 4400 50  0000 L CNN
-F 1 "2.2uF 0603 16V" V 7675 3925 50  0000 L CNN
-F 2 "Capacitor_SMD:C_0603_1608Metric" H 7563 4175 50  0001 C CNN
+F 1 "2.2uF 0402 16V" V 7675 3925 50  0000 L CNN
+F 2 "Capacitor_SMD:C_0402_1005Metric" H 7563 4175 50  0001 C CNN
 F 3 "~" H 7525 4325 50  0001 C CNN
 	1    7525 4325
@@
 AR Path="/61017570/6101FE0E" Ref="C603"  Part="1"
 F 0 "C603" H 5117 3921 50  0000 L CNN
-F 1 "1uF 0603 16V" H 4450 3950 50  0000 L CNN
-F 2 "Capacitor_SMD:C_0603_1608Metric" H 5025 3875 50  0001 C CNN
+F 1 "1uF 0402 16V" H 4450 3950 50  0000 L CNN
+F 2 "Capacitor_SMD:C_0402_1005Metric" H 5025 3875 50  0001 C CNN
 F 3 "~" H 5025 3875 50  0001 C CNN
 	1    5025 3875
@@
 AR Path="/61017570/6101FF32" Ref="C604"  Part="1"
 F 0 "C604" H 5117 4271 50  0000 L CNN
-F 1 "1uF 0603 16V" H 4450 4300 50  0000 L CNN
-F 2 "Capacitor_SMD:C_0603_1608Metric" H 5025 4225 50  0001 C CNN
+F 1 "1uF 0402 16V" H 4450 4300 50  0000 L CNN
+F 2 "Capacitor_SMD:C_0402_1005Metric" H 5025 4225 50  0001 C CNN
 F 3 "~" H 5025 4225 50  0001 C CNN
 	1    5025 4225
@@
 P 6875 4325
 F 0 "C605" V 6825 4400 50  0000 L CNN
-F 1 "2.2uF 0603 16V" V 7025 3925 50  0000 L CNN
-F 2 "Capacitor_SMD:C_0603_1608Metric" H 6913 4175 50  0001 C CNN
+F 1 "2.2uF 0402 16V" V 7025 3925 50  0000 L CNN
+F 2 "Capacitor_SMD:C_0402_1005Metric" H 6913 4175 50  0001 C CNN
 F 3 "~" H 6875 4325 50  0001 C CNN
 	1    6875 4325
@@
 Wire Wire Line
 	5775 2775 5775 2625
+$Comp
+L power:+3.3V #PWR0155
+U 1 1 613A2FC1
+P 4750 3675
+F 0 "#PWR0155" H 4750 3525 50  0001 C CNN
+F 1 "+3.3V" H 4765 3848 50  0000 C CNN
+F 2 "" H 4750 3675 50  0001 C CNN
+F 3 "" H 4750 3675 50  0001 C CNN
+	1    4750 3675
+	1    0    0    -1
+$EndComp
+Wire Wire Line
+	4750 3675 5325 3675
 $EndSCHEMATC
